File: PowerSupply.kicad_pcb (KiCad board)
At the start: 2 copper layers, 50 x 50 mm, 35 parts, among them CN1 SM04B-SRSS-TB (LF)(SN), Q1 CSD17318Q2, Q2 CSD17318Q2, U1 TPS55288RPMR

Commit message: Removed TP
Parts:
- moved C314 12.9 mm to (60.5, 52.3)
- moved U1 5.18 mm to (67.0, 56.1)
Changed lines of the file:
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@@
 	(footprint "easyeda2kicad:C0603"
 		(layer "F.Cu")
-		(at 63 65 90)
+		(at 60.5 52.32 90)
 		(property "Reference" "C314"
 			(at 0 -2 90)
@@
 	(footprint "easyeda2kicad:VQFN-HR-26_L4.0-W3.5_TPS55288RPMR"
 		(layer "F.Cu")
-		(at 69.84 60.5)
+		(at 67.05 56.14)
 		(property "Reference" "U1"
 			(at 0 -5.79 0)
